Commit message: lite: urdf done

File: src/misc/roar-urdf/src/gokart/_perceptions.urdf (robot description, URDF)
Before this commit: robot gokart, 1 links, 1 joints
Links:
- added link zed; visual mesh filename=file://$(find roar-urdf)/meshes/ZED2i.stl scale=0.001 0.001 0.001
Joints:
- added joint zed2i: type fixed, parent center_lidar, child zed, origin xyz=0.0 0 0.1 rpy=0 0 0

Commit message: zed -> camera

File: src/misc/roar-urdf/src/gokart/_perceptions.urdf (robot description, URDF)
Before this commit: robot gokart, 2 links, 2 joints
Links:
- removed link zed
- added link camera; visual mesh filename=file://$(find roar-urdf)/meshes/ZED2i.stl scale=0.001 0.001 0.001
Joints:
- removed joint zed2i
- added joint camera: type fixed, parent center_lidar, child camera, origin xyz=0.0 0 0.1 rpy=0 0 0
