Commit message: lite: global planner done

File: src/misc/roar-urdf/src/gokart/_gnss.urdf (robot description, URDF)
Before this commit: robot gokart, 2 links, 2 joints
Links:
- removed link gps_antenna
- added link gnss; visual mesh filename=file://$(find roar-urdf)/meshes/gps_antenna.stl scale=0.001 0.001 0.001
Joints:
- removed joint gps_antenna_joint
- added joint gnss_joint: type fixed, parent gps_platform, child gnss, origin xyz=0 0 0.1 rpy=0 0 0
